Commit message: changed friction coefficient to make the caster wheel slip on the ground driving wheel are not having high coefficient to ensure traction

File: src/merlin_description/urdf/merlin.urdf.xacro (robot description, xacro)
@@ -6,5 +6,5 @@
   <xacro:include filename="$(find merlin_description)/urdf/materials.xacro" />
   <link name="world"/>
-  <joint name="fixed" type="fixed">
+  <joint name="fixed" type="floating">
     <parent link="world"/>
     <child link="base_link"/>
@@ -53,4 +53,5 @@
     <origin xyz="0 0.115 0.046" rpy="1.5708 0 0"/>
     <axis xyz="0 0 1"/>
+    <dynamics damping="0.7"/>
   </joint>
   <link name="rwheel">
@@ -80,4 +81,5 @@
     <origin xyz="0 -0.115 0.046" rpy="-1.5708 0 0"/>
     <axis xyz="0 0 1"/>
+    <dynamics damping="0.7"/>
   </joint>
   <link name="fwheel_attach">
@@ -106,4 +108,5 @@
     <child link="fwheel_attach"/>
     <origin xyz="0 0 0" rpy="0 0 0"/>
+    <axis xyz="0 0 1"/>
   </joint>
   <link name="fwheel">
@@ -128,8 +131,9 @@
     </inertial>
   </link>
-  <joint name="base_to_fwheel" type="continuous">
+  <joint name="base_to_fwheel" type="fixed">
     <parent link="base_link"/>
     <child link="fwheel"/>
     <origin xyz="0.13 0 0.02" rpy="0 0 0"/>
+    <axis xyz="0 1 0"/>
   </joint>
    <transmission name="tran1">

Commit message: flipped wheel so platform can be moved with cmd_vel inertia is too low which causes the platform to jerk

File: src/merlin_description/urdf/merlin.urdf.xacro (robot description, xacro)
@@ -2,5 +2,5 @@
 <robot name="merlin" xmlns:xacro="http://www.ros.org/wiki/xacro">
   <xacro:property name="PI" value="3.1415926535897931"/>
-  <xacro:property name="mass" value="1"/>
+  <xacro:property name="mass" value="10"/>
   <xacro:include filename="$(find merlin_description)/urdf/merlin.gazebo" />
   <xacro:include filename="$(find merlin_description)/urdf/materials.xacro" />
@@ -79,5 +79,5 @@
     <parent link="base_link"/>
     <child link="rwheel"/>
-    <origin xyz="0 -0.115 0.046" rpy="-1.5708 0 0"/>
+    <origin xyz="0 -0.115 0.046" rpy="1.5708 0 0"/>
     <axis xyz="0 0 1"/>
     <dynamics damping="0.7"/>

Commit message: changes to inertia

File: src/merlin_description/urdf/merlin.urdf.xacro (robot description, xacro)
@@ -2,5 +2,5 @@
 <robot name="merlin" xmlns:xacro="http://www.ros.org/wiki/xacro">
   <xacro:property name="PI" value="3.1415926535897931"/>
-  <xacro:property name="mass" value="10"/>
+  <xacro:property name="mass" value="50"/>
   <xacro:include filename="$(find merlin_description)/urdf/merlin.gazebo" />
   <xacro:include filename="$(find merlin_description)/urdf/materials.xacro" />
@@ -26,5 +26,5 @@
     <inertial>
       <mass value="${mass}"/>
-      <inertia ixx="0.4" ixy="0.0" ixz="0.0" iyy="0.4" iyz="0.0" izz="0.2"/>
+      <inertia ixx="10.4" ixy="0.0" ixz="0.0" iyy="10.4" iyz="0.0" izz="10.2"/>
     </inertial>
   </link>

Commit message: able to launch multiple robot need to change the main launchfile gazebo plugin does not launch after the first robot

File: src/merlin_description/urdf/merlin.urdf.xacro (robot description, xacro)
@@ -1,7 +1,29 @@
 <?xml version="1.0"?>
-<robot name="merlin" xmlns:xacro="http://www.ros.org/wiki/xacro">
+<robot name="$(arg robot_name)" xmlns:xacro="http://www.ros.org/wiki/xacro">
   <xacro:property name="PI" value="3.1415926535897931"/>
   <xacro:property name="mass" value="50"/>
-  <xacro:include filename="$(find merlin_description)/urdf/merlin.gazebo" />
+  <gazebo>
+    <plugin name="gazebo_ros_control" filename="libgazebo_ros_control.so">
+      <robotNamespace>$(arg robot_name)</robotNamespace>
+      <robotSimType>gazebo_ros_control/DefaultRobotHWSim</robotSimType>
+    </plugin>
+  </gazebo>
+  <gazebo reference="base_link">
+    <material>Gazebo/Orange</material>
+  </gazebo>
+  <gazebo reference="rwheel">
+    <mu1>200.2</mu1>
+    <mu2>200.2</mu2>
+    <material>Gazebo/Black</material>
+  </gazebo>
+  <gazebo reference="lwheel">
+    <mu1>200.2</mu1>
+    <mu2>200.2</mu2>
+    <material>Gazebo/Black</material>
+  </gazebo>
+  <gazebo reference="fwheel">
+    <mu1>0.0001</mu1>
+    <mu2>0.0001</mu2>
+  </gazebo>
   <xacro:include filename="$(find merlin_description)/urdf/materials.xacro" />
   <link name="world"/>

Commit message: integrated fake localization

File: src/merlin_description/urdf/merlin.urdf.xacro (robot description, xacro)
@@ -73,5 +73,5 @@
     <parent link="base_link"/>
     <child link="lwheel"/>
-    <origin xyz="0 0.115 0.046" rpy="1.5708 0 0"/>
+    <origin xyz="0 -0.115 0.046" rpy="1.5708 0 0"/>
     <axis xyz="0 0 1"/>
     <dynamics damping="0.7"/>
@@ -101,5 +101,5 @@
     <parent link="base_link"/>
     <child link="rwheel"/>
-    <origin xyz="0 -0.115 0.046" rpy="1.5708 0 0"/>
+    <origin xyz="0 0.115 0.046" rpy="1.5708 0 0"/>
     <axis xyz="0 0 1"/>
     <dynamics damping="0.7"/>

Commit message: add navigation with spot turn nav.py added start_path in path_store to trigger navigation given path name and robot name flipped robot urdf to correspond with gazebo frame when moving forward multiple robot navigation possible

File: src/merlin_description/urdf/merlin.urdf.xacro (robot description, xacro)
@@ -73,5 +73,5 @@
     <parent link="base_link"/>
     <child link="lwheel"/>
-    <origin xyz="0 -0.115 0.046" rpy="1.5708 0 0"/>
+    <origin xyz="0 0.115 0.046" rpy="1.5708 0 3.14"/>
     <axis xyz="0 0 1"/>
     <dynamics damping="0.7"/>
@@ -101,5 +101,5 @@
     <parent link="base_link"/>
     <child link="rwheel"/>
-    <origin xyz="0 0.115 0.046" rpy="1.5708 0 0"/>
+    <origin xyz="0 -0.115 0.046" rpy="1.5708 0 3.14"/>
     <axis xyz="0 0 1"/>
     <dynamics damping="0.7"/>
@@ -110,5 +110,5 @@
         <cylinder length="0.060" radius="0.023"/>
       </geometry>
-      <origin rpy="0 0 0" xyz="0.13 0 0.08"/>
+      <origin rpy="0 0 0" xyz="-0.13 0 0.08"/>
       <material name="white">
         <color rgba="1 1 1 1"/>
@@ -156,5 +156,5 @@
     <parent link="base_link"/>
     <child link="fwheel"/>
-    <origin xyz="0.13 0 0.02" rpy="0 0 0"/>
+    <origin xyz="-0.13 0 0.02" rpy="0 0 0"/>
     <axis xyz="0 1 0"/>
   </joint>
